File: diodyled.kicad_sch (KiCad schematic)
At the start: 34 parts

Commit message: Poprawiono wygląd schematu
Parts:
- removed C18, C19, C20, C21, C22, C23, C24, C25, C26, C27, C29, C30, C31, C32, C33, C34: 100n, Capacitor_SMD:C_0402_1005Metric, symbol Device:C
- added C18, C19, C20, C21, C22, C23, C24, C25, C26, C27, C29, C30, C31, C32, C33, C34: 100n, Capacitor_SMD:C_0402_1005Metric, symbol Device:C_Small
- C28: symbol Device:C -> Device:C_Small
Connections:
- net +5V: now also C18.2, C19.2, C20.2, C21.2, C22.2, C23.2, C24.2, C25.2, C26.2, C27.2, C29.2, C30.2, C31.2, C32.2, C33.2, C34.2
- net GND: now also C18.1, C19.1, C20.1, C21.1, C22.1, C23.1, C24.1, C25.1, C26.1, C27.1, C29.1, C30.1, C31.1, C32.1, C33.1, C34.1
- net LED_Data1: now reaches LED12.2 (DOUT), LED13.4 (DIN)
- net LED_Data0: now reaches LED6.2 (DOUT), LED7.4 (DIN)
Other:
- moved on the sheet: C28
